Commit message: Before starting to integrating dual-arm redunancy main algorithm, current progress loads the dual arm frnka with grippers and attaches to the table.

File: src/gazebo_assets/table.urdf (robot description, URDF)
Before this commit: robot table, 1 links, 0 joints
Links:
- link table_link: geometry collision mesh filename=package://gazebo_assets/meshes/table.stl scale=0.0005 0.0005 0.0005; visual mesh filename=package://gazebo_assets/meshes/table.stl scale=0.0005 0.0005 0.0005

File: src/panda_multiple_arms/robot_description/panda_multiple_arms.xacro (robot description, xacro)
@@ -12,7 +12,7 @@
     <link name="base">
         <visual>
-            <origin xyz="0 0 0.5" rpy="0 0 0" />
+            <origin xyz="0 0 0.0" rpy="0 0 0" />
             <geometry>
-                <box size="1 2 1" />
+                <box size="0 0 0" />
             </geometry>
             <material name="White">
@@ -21,12 +21,12 @@
         </visual>
         <collision>
-            <origin xyz="0 0 0.5" rpy="0 0 0" />
+            <origin xyz="0 0 0.0" rpy="0 0 0" />
             <geometry>
-                <box size="1 2 1" />
+                <box size="0 0 0" />
             </geometry>
         </collision>
         <inertial>
             <origin xyz="0.0 0.0 0.0" rpy="0.0 0.0 0.0"/>
-            <mass value="10.0"/>
+            <mass value="0.01"/>
             <inertia ixx="0.001" ixy="0.0" ixz="0.001" iyy="0.0" iyz="0.0" izz="0.001"/>
         </inertial>
@@ -38,8 +38,8 @@
     </joint>
     <!-- right arm with gripper -->
-    <xacro:franka_arm arm_id="$(arg arm_id_1)" connected_to="base" xyz="0 -0.25 1" gazebo="true" safety_distance="0.03" joint_limits="${xacro.load_yaml('$(find franka_description)/robots/panda/joint_limits.yaml')}"/>
+    <xacro:franka_arm arm_id="$(arg arm_id_1)" connected_to="base" xyz="0 -0.25 0" gazebo="true" safety_distance="0.03" joint_limits="${xacro.load_yaml('$(find franka_description)/robots/panda/joint_limits.yaml')}"/>
     <xacro:franka_hand arm_id="$(arg arm_id_1)" rpy="0 0 ${-pi/4}" connected_to="$(arg arm_id_1)_link8" gazebo="true" safety_distance="0.03" />
     <!-- left arm with gripper -->
-    <xacro:franka_arm arm_id="$(arg arm_id_2)" connected_to="base" xyz="0 0.25 1" gazebo="true" safety_distance="0.03" joint_limits="${xacro.load_yaml('$(find franka_description)/robots/panda/joint_limits.yaml')}"/>
+    <xacro:franka_arm arm_id="$(arg arm_id_2)" connected_to="base" xyz="0 0.25 0" gazebo="true" safety_distance="0.03" joint_limits="${xacro.load_yaml('$(find franka_description)/robots/panda/joint_limits.yaml')}"/>
     <xacro:franka_hand arm_id="$(arg arm_id_2)" rpy="0 0 ${-pi/4}" connected_to="$(arg arm_id_2)_link8" gazebo="true" safety_distance="0.03" />
     <!-- right arm joints control interface -->
