Commit message: Changes made during the IISc Experimental Validation.

File: src/without_gripper_panda_multiple_arms/robot_description/panda_multiple_arms.xacro (robot description, xacro)
@@ -13,5 +13,5 @@
             <origin xyz="0 0 0.5" rpy="0 0 0" />
             <geometry>
-                <box size="1 2 1" />
+                <box size="1.6 1.75 1" />
             </geometry>
             <material name="White">
@@ -37,7 +37,7 @@
     </joint>
     <!-- right arm without gripper -->
-    <xacro:franka_arm arm_id="$(arg arm_id_1)" connected_to="base" xyz="0 -0.20 1" gazebo="true" safety_distance="0.03" joint_limits="${xacro.load_yaml('$(find franka_description)/robots/panda/joint_limits.yaml')}"/>
+    <xacro:franka_arm arm_id="$(arg arm_id_1)" connected_to="base" xyz="0 -0.50 1" rpy="0 0 1.571" gazebo="true" safety_distance="0.03" joint_limits="${xacro.load_yaml('$(find franka_description)/robots/panda/joint_limits.yaml')}"/>
     <!-- left arm without gripper -->
-    <xacro:franka_arm arm_id="$(arg arm_id_2)" connected_to="base" xyz="0 0.20 1" gazebo="true" safety_distance="0.03" joint_limits="${xacro.load_yaml('$(find franka_description)/robots/panda/joint_limits.yaml')}"/>
+    <xacro:franka_arm arm_id="$(arg arm_id_2)" connected_to="base" xyz="0 0.50 1" rpy="0 0 -1.571" gazebo="true" safety_distance="0.03" joint_limits="${xacro.load_yaml('$(find franka_description)/robots/panda/joint_limits.yaml')}"/>
     <!-- right arm joints control interface -->
     <xacro:gazebo-joint joint="$(arg arm_id_1)_joint1" transmission="hardware_interface/PositionJointInterface" />
